Commit message: Feat: urdf accessories update

File: rdsim_description/urdf/accessories/bridge_plate.urdf.xacro (robot description, xacro)
@@ -17,5 +17,5 @@
         <origin xyz="0 0 0" rpy="1.5707 0.0 1.5707" />
         <geometry>
-          <mesh filename="file://$(find rdsim_description)/meshes/bridge_plate.stl" scale="0.001 0.001 0.001" />
+          <mesh filename="file://$(find rdsim_description)/meshes/bridge-plate.stl" scale="0.001 0.001 0.001" />
         </geometry>
         <material name="dark_grey" />

File: rdsim_description/urdf/accessories/camera_mount.urdf.xacro (robot description, xacro)
@@ -5,5 +5,5 @@
         <origin xyz="0 0 0" rpy="1.5707 0 1.5707" />
         <geometry>
-          <mesh filename="file://$(find rdsim_description)/meshes/camera_mount.stl" scale="0.001 0.001 0.001" />
+          <mesh filename="file://$(find rdsim_description)/meshes/camera-mount.stl" scale="0.001 0.001 0.001" />
         </geometry>
         <material name="dark_grey" />
@@ -14,5 +14,5 @@
         <origin xyz="0 0 0" rpy="0 0 1.5707" />
         <geometry>
-          <mesh filename="file://$(find rdsim_description)/meshes/camera_beam.stl" scale="0.001 0.001 0.001" />
+          <mesh filename="file://$(find rdsim_description)/meshes/camera-beam.stl" scale="0.001 0.001 0.001" />
         </geometry>
         <material name="dark_grey" />

File: rdsim_description/urdf/accessories/hokuyo_ust10.urdf.xacro (robot description, xacro)
@@ -61,5 +61,5 @@
         <geometry>
           <!-- Origin of this mesh is the base of the bracket. -->
-          <mesh filename="file://$(find rdsim_description)/meshes/hokuyo_ust10_mount.stl" />
+          <mesh filename="file://$(find rdsim_description)/meshes/hokuyo_ust10.stl" />
         </geometry>
         <material name="dark_grey" />

File: rdsim_description/urdf/accessories/sick_lms1xx_mount.urdf.xacro (robot description, xacro)
@@ -39,5 +39,5 @@
         <geometry>
           <!-- Origin of this mesh is the base of the bracket. -->
-          <mesh filename="file://$(find rdsim_description)/meshes/sick_lms1xx_mount.stl" scale="0.001 0.001 0.001" />
+          <mesh filename="file://$(find rdsim_description)/meshes/sick-lms1xx-bracket.stl" scale="0.001 0.001 0.001" />
         </geometry>
         <material name="dark_grey" />
