Commit message: Fix: 3D LiDAR translation modify

File: rdsim_description/urdf/accessories/vlp16_mount.urdf.xacro (robot description, xacro)
@@ -60,5 +60,5 @@
       <parent link="${parent_link}" />
       <child link="${prefix}_vlp16_mount" />
-      <origin xyz="0.15 0.05 0.17" rpy="0 0.436332 0" />
+      <origin xyz="0.15 0 0.17" rpy="0 0.436332 0" />
       <xacro:insert_block name="origin" />
     </joint>
