Commit message: Feat: Gazebo sensor(2D LiDAR x2, 3D LiDAR x1, RGBD Camera x1) add

File: rdsim_description/urdf/accessories.urdf.xacro (robot description, xacro)
@@ -26,7 +26,7 @@
   -->
   <!-- Primary 2D Lidar -->
-  <xacro:if value="$(optenv JACKAL_LASER 0)">
+  <xacro:if value="$(optenv JACKAL_LASER 1)">
     <xacro:property name="mount" value="$(optenv JACKAL_LASER_MOUNT front)" />
-    <xacro:property name="topic" value="$(optenv JACKAL_LASER_TOPIC front/scan)" />
+    <xacro:property name="topic" value="$(optenv JACKAL_LASER_TOPIC scan/front)" />
     <xacro:property name="tower" value="$(optenv JACKAL_LASER_TOWER 1)" />
     <xacro:property name="prefix" value="$(optenv JACKAL_LASER_PREFIX ${mount})" />
@@ -60,12 +60,12 @@
     <xacro:if value="${lidar_model == 'ust10'}">
       <xacro:hokuyo_ust10_mount topic="${topic}" prefix="${prefix}" parent_link="${parent}">
-        <origin xyz="$(optenv JACKAL_LASER_OFFSET 0 0 0)" rpy="$(optenv JACKAL_LASER_RPY 0 0 0)" />
+        <origin xyz="$(optenv JACKAL_LASER_OFFSET 0.11 0 -0.17)" rpy="$(optenv JACKAL_LASER_RPY 0 0 0)" />
       </xacro:hokuyo_ust10_mount>
     </xacro:if>
   </xacro:if>
   <!-- Secondary 2D Lidar -->
-  <xacro:if value="$(optenv JACKAL_LASER_SECONDARY 0)">
+  <xacro:if value="$(optenv JACKAL_LASER_SECONDARY 1)">
     <xacro:property name="mount" value="$(optenv JACKAL_LASER_SECONDARY_MOUNT rear)" />
-    <xacro:property name="topic" value="$(optenv JACKAL_LASER_SECONDARY_TOPIC rear/scan)" />
+    <xacro:property name="topic" value="$(optenv JACKAL_LASER_SECONDARY_TOPIC scan/rear)" />
     <xacro:property name="tower" value="$(optenv JACKAL_LASER_SECONDARY_TOWER 1)" />
     <xacro:property name="prefix" value="$(optenv JACKAL_LASER_SECONDARY_PREFIX ${mount})" />
@@ -99,5 +99,5 @@
     <xacro:if value="${lidar_model == 'ust10'}">
       <xacro:hokuyo_ust10_mount topic="${topic}" prefix="${prefix}" parent_link="${parent}">
-        <origin xyz="$(optenv JACKAL_LASER_SECONDARY_OFFSET 0 0 0)" rpy="$(optenv JACKAL_LASER_SECONDARY_RPY 0 0 3.14159)" />
+        <origin xyz="$(optenv JACKAL_LASER_SECONDARY_OFFSET -0.11 0 -0.17)" rpy="$(optenv JACKAL_LASER_SECONDARY_RPY 0 0 3.14159)" />
       </xacro:hokuyo_ust10_mount>
     </xacro:if>
@@ -109,5 +109,5 @@
     - vlp32e           :: Velodyne HDL-32E
   -->
-  <xacro:if value="$(optenv JACKAL_LASER_3D 0)">
+  <xacro:if value="$(optenv JACKAL_LASER_3D 1)">
     <xacro:property name="mount" value="$(optenv JACKAL_LASER_3D_MOUNT mid)" />
     <xacro:property name="topic" value="$(optenv JACKAL_LASER_3D_TOPIC mid/points)" />
@@ -118,14 +118,14 @@
     <!-- Velodyne VLP16 -->
     <xacro:if value="${lidar_3d_model == 'vlp16'}">
-      <xacro:vlp16_mount topic="${topic}" tower="${tower}" prefix="${prefix}" parent_link="${parent}" >
+      <xacro:vlp16_mount topic="${topic}" prefix="${prefix}" parent_link="${parent}" >
         <origin xyz="$(optenv JACKAL_LASER_3D_OFFSET 0 0 0)" rpy="$(optenv JACKAL_LASER_3D_RPY 0 0 0)" />
       </xacro:vlp16_mount>
     </xacro:if>
     <!-- Velodyne HDL-32E -->
-    <xacro:if value="${lidar_3d_model == 'hdl32e'}">
+    <!-- <xacro:if value="${lidar_3d_model == 'hdl32e'}">
       <xacro:hdl32e_mount topic="${topic}" tower="${tower}" prefix="${prefix}" parent_link="${parent}" >
         <origin xyz="$(optenv JACKAL_LASER_3D_OFFSET 0 0 0)" rpy="$(optenv JACKAL_LASER_3D_RPY 0 0 0)" />
       </xacro:hdl32e_mount>
-    </xacro:if>
+    </xacro:if> -->
   </xacro:if>
   <!--

File: rdsim_description/urdf/accessories/hokuyo_ust10.urdf.xacro (robot description, xacro)
@@ -39,5 +39,5 @@
             </noise>
           </ray>
-          <plugin name="gazebo_ros_laser" filename="libgazebo_ros_ray_sensor.so">
+          <plugin name="${prefix}_gazebo_ros_laser" filename="libgazebo_ros_ray_sensor.so">
             <ros>
               <namespace>${robot_namespace}</namespace>

File: rdsim_description/urdf/accessories/vlp16_mount.urdf.xacro (robot description, xacro)
@@ -1,4 +1,5 @@
+<?xml version="1.0"?>
 <robot xmlns:xacro="http://wiki.ros.org/xacro">
-  <xacro:include filename="$(find velodyne_description)/urdf/VLP-16.urdf.xacro" />
+  <xacro:include filename="$(find rdsim_description)/urdf/accessories/VLP-16.urdf.xacro" />
   <xacro:macro name="vlp16_mount" params="prefix parent_link topic height:=0.1 *origin">
     <link name="${prefix}_vlp16_mount" />
@@ -6,5 +7,5 @@
       <visual>
         <geometry>
-          <box size="0.1 0.1 0.002" />
+          <box size="0.11 0.1 0.002" />
         </geometry>
         <material name="black" />
@@ -12,5 +13,5 @@
       </visual>
     </link>
-    <link name="${prefix}_vlp16_leg1">
+    <!-- <link name="${prefix}_vlp16_leg1">
       <visual>
         <geometry>
@@ -55,11 +56,12 @@
         <origin xyz="0 0 ${height/2}" rpy="0 0 0" />
       </visual>
-    </link>
+    </link> -->
     <joint name="${prefix}_vlp16_mount_joint" type="fixed">
       <parent link="${parent_link}" />
       <child link="${prefix}_vlp16_mount" />
+      <origin xyz="0.15 0.05 0.17" rpy="0 0.436332 0" />
       <xacro:insert_block name="origin" />
     </joint>
-    <joint name="${prefix}_vlp16_leg1_joint" type="fixed">
+    <!-- <joint name="${prefix}_vlp16_leg1_joint" type="fixed">
       <parent link="${prefix}_mount" />
       <child link="${prefix}_vlp16_leg1" />
@@ -80,5 +82,5 @@
       <child link="${prefix}_vlp16_leg4" />
       <origin xyz="-0.05 -0.05 0" rpy="0 0 0" />
-    </joint>
+    </joint> -->
     <joint name="${prefix}_vlp16_plate_joint" type="fixed">
       <parent link="${prefix}_vlp16_mount" />

File: rdsim_description/urdf/jackal.urdf.xacro (robot description, xacro)
@@ -225,4 +225,34 @@
     <origin xyz="${mount_spacing} 0 0" />
   </joint>
+  <!-- AuTURBO modify -->
+  <link name="food_storage_link">
+    <visual>
+      <geometry>
+        <box size="0.4 0.3 0.3" />
+      </geometry>
+      <material name="yellow" />
+    </visual>
+  </link>
+  <joint name="food_storage_joint" type="fixed">
+    <parent link="mid_mount" />
+    <child link="food_storage_link" />
+    <origin xyz="0 0 0.125" />
+  </joint>
+  <link name="front_camera_link">
+    <visual>
+      <geometry>
+        <box size="0.01 0.05 0.02" />
+      </geometry>
+      <material name="yellow" />
+    </visual>
+  </link>
+  <joint name="front_camera_joint" type="fixed">
+    <parent link="mid_mount" />
+    <child link="front_camera_link" />
+    <origin xyz="0.2 0 0.15" />
+  </joint>
+  <!-- CAMERA -->
+  <xacro:include filename="$(find rdsim_description)/urdf/accessories/kinect_camera.urdf.xacro" />
+  <xacro:kinect_camera />
   <!-- ROS2 controls -->
   <ros2_control name="jackal_hardware" type="system">

File: velodyne_simulator/velodyne_description/urdf/example.urdf.xacro (robot description, xacro)
@@ -14,10 +14,10 @@
     <visual>
       <geometry>
-        <box size="0.5 0.5 0.1" />
+        <box size="0.5 0.5 0.5" />
       </geometry>
     </visual>
     <collision>
       <geometry>
-        <box size="0.5 0.5 0.1" />
+        <box size="0.5 0.5 0.5" />
       </geometry>
     </collision>
@@ -34,5 +34,5 @@
     <origin xyz="0 0 0.4" rpy="0 0 0" />
   </VLP-16>
-  <xacro:include filename="$(find velodyne_description)/urdf/HDL-32E.urdf.xacro"/>
+  <!-- <xacro:include filename="$(find velodyne_description)/urdf/HDL-32E.urdf.xacro"/>
    <HDL-32E parent="base_link" name="velodyne2" topic="/velodyne_points2" hz="10" samples="220" gpu="${gpu}">
     <origin xyz="0 0 0.6" rpy="0 0 0" />
@@ -41,4 +41,4 @@
   <VLP-32C parent="base_link" name="velodyne3" topic="/velodyne_points3" hz="10" samples="1200" gpu="${gpu}">
     <origin xyz="0 0 0.8" rpy="0 0 0" />
-  </VLP-32C>
+  </VLP-32C> -->
 </robot>
