Commit message: Feat: Jackal Controller devel and Gazebo robot spwan base function clear

File: rdsim_description/urdf/jackal.urdf.xacro (robot description, xacro)
@@ -94,5 +94,5 @@
       <origin xyz="0 0 ${footprint_vertical_offset}" rpy="${PI/2} 0 ${PI/2}"/>
       <geometry>
-        <mesh filename="file://$(find rdsim_description)/meshes/jackal-chassis.stl"/>
+        <mesh filename="file://$(find rdsim_description)/meshes/jackal-base.stl"/>
       </geometry>
       <material name="dark_grey" />
@@ -265,4 +265,6 @@
        default each one to off.-->
   <xacro:include filename="$(find rdsim_description)/urdf/accessories.urdf.xacro" />
+  <!-- 물성치 -->
+  <xacro:include filename="$(find rdsim_description)/urdf/jackal.gazebo.xacro" />
   <!-- Optional custom includes. -->
   <xacro:include filename="$(optenv JACKAL_URDF_EXTRAS empty.urdf)" />

Commit message: Feat: follow camera(top view) add

File: rdsim_description/urdf/jackal.urdf.xacro (robot description, xacro)
@@ -239,17 +239,7 @@
     <origin xyz="0 0 0.125" />
   </joint>
-  <link name="front_camera_link">
-    <visual>
-      <geometry>
-        <box size="0.01 0.05 0.02" />
-      </geometry>
-      <material name="yellow" />
-    </visual>
-  </link>
-  <joint name="front_camera_joint" type="fixed">
-    <parent link="mid_mount" />
-    <child link="front_camera_link" />
-    <origin xyz="0.2 0 0.15" />
-  </joint>
+  <!-- Follow camera-->
+  <xacro:include filename="$(find rdsim_description)/urdf/accessories/follow_camera.urdf.xacro" />
+  <xacro:follow_camera />
   <!-- CAMERA -->
   <xacro:include filename="$(find rdsim_description)/urdf/accessories/kinect_camera.urdf.xacro" />
