Commit message: fix : lidar tf 수정

File: rdsim_description/urdf/rdsim.urdf.xacro (robot description, xacro)
@@ -193,5 +193,5 @@
     <parent link="base_link"/>
     <child link="lidar_link"/>
-    <origin xyz="0 0 0.24" rpy="0 0 0"/>
+    <origin xyz="0 0 0.44" rpy="0 0 0"/>
   </joint>
   <link name="camera_link">
