Commit message: feat : gps 기능 추가

File: rdsim_description/urdf/rdsim.gazebo.xacro (robot description, xacro)
@@ -237,3 +237,30 @@
     </sensor>
   </gazebo>
+  <!-- GPS -->
+  <gazebo reference="gps_link">
+    <sensor name="gps_sensor" type="gps">
+      <plugin filename="libgazebo_ros_gps_sensor.so" name="gps_plugin">
+        <ros>
+          <namespace>/gps</namespace>
+          <remapping>~/out:=gps/data</remapping>
+        </ros>
+        <output_type>sensor_msgs/NavSatFix</output_type>
+        <frame_name>gps_link</frame_name>
+        <!-- 임의의 위도, 경도 값 설정 -->
+        <latitude_deg>37.466</latitude_deg>
+        <longitude_deg>126.932</longitude_deg>
+        <altitude>0.0</altitude>
+      </plugin>
+      <always_on>true</always_on>
+      <update_rate>10</update_rate>
+      <gps>
+        <position_sensing>
+          <noise type="gaussian">
+            <mean>0.0</mean> <!-- 기본적으로 노이즈가 없는 설정 -->
+            <stddev>0.0</stddev> <!-- 노이즈 표준편차 설정 -->
+          </noise>
+        </position_sensing>
+      </gps>
+    </sensor>
+  </gazebo>
 </robot>

File: rdsim_description/urdf/rdsim.urdf.xacro (robot description, xacro)
@@ -59,4 +59,18 @@
     <xacro:box_inertia m="15" w="${base_width}" d="${base_length}" h="${base_height}"/>
   </link>
+<!-- gps link -->
+  <link name="gps_link">
+    <visual>
+      <geometry>
+        <box size="0.001 0.001 0.001"/>
+      </geometry>
+    </visual>
+  </link>
+  <!-- gps joint -->
+  <joint name="gps_joint" type="fixed">
+    <parent link="base_footprint"/>
+    <child link="gps_link"/>
+    <origin xyz="0 0 0.01"/>
+  </joint>
   <link name="wheel_left_link">
     <visual>

Commit message: feat : ouster fov 늘림

File: rdsim_description/urdf/rdsim.gazebo.xacro (robot description, xacro)
@@ -216,6 +216,6 @@
             <samples>32</samples> <!-- 수직 샘플 수 줄임 -->
             <resolution>1</resolution>
-            <min_angle>-0.261799</min_angle>
-            <max_angle>0.261799</max_angle>
+            <min_angle>-0.561799</min_angle>
+            <max_angle>0.561799</max_angle>
           </vertical>
         </scan>

File: rdsim_description/urdf/rdsim.urdf.xacro (robot description, xacro)
@@ -141,5 +141,5 @@
     <parent link="base_link"/>
     <child link="caster_link"/>
-    <origin xyz="${-caster_xoff} 0.0 ${-(base_height)-0.005}" rpy="0 0 0"/>
+    <origin xyz="${-caster_xoff} 0.0 ${-(base_height)-0.015}" rpy="0 0 0"/>
   </joint>
   <link name="imu_link">

Commit message: feat : 4축 camera setting 완료

File: rdsim_description/urdf/rdsim.gazebo.xacro (robot description, xacro)
@@ -264,3 +264,108 @@
     </sensor>
   </gazebo>
+<!-- 카메라 플러그인 추가 -->
+<!-- Front-right camera -->
+<gazebo reference="camera_front_right_link">
+  <sensor type="camera" name="camera_front_right_sensor">
+    <always_on>true</always_on>
+    <update_rate>30.0</update_rate>
+    <camera>
+      <horizontal_fov>1.047</horizontal_fov>
+      <image>
+        <width>640</width>
+        <height>480</height>
+        <format>R8G8B8</format>
+      </image>
+      <clip>
+        <near>0.02</near>
+        <far>50.0</far>
+      </clip>
+    </camera>
+    <plugin name="camera_front_right_controller" filename="libgazebo_ros_camera.so">
+      <ros>
+        <namespace>camera_front_right</namespace>
+        <remapping>image_raw:=/camera_front_right/image_raw</remapping>
+        <remapping>camera_info:=/camera_front_right/camera_info</remapping>
+      </ros>
+    </plugin>
+  </sensor>
+</gazebo>
+<!-- Front-left camera -->
+<gazebo reference="camera_front_left_link">
+  <sensor type="camera" name="camera_front_left_sensor">
+    <always_on>true</always_on>
+    <update_rate>30.0</update_rate>
+    <camera>
+      <horizontal_fov>1.047</horizontal_fov>
+      <image>
+        <width>640</width>
+        <height>480</height>
+        <format>R8G8B8</format>
+      </image>
+      <clip>
+        <near>0.02</near>
+        <far>50.0</far>
+      </clip>
+    </camera>
+    <plugin name="camera_front_left_controller" filename="libgazebo_ros_camera.so">
+      <ros>
+        <namespace>camera_front_left</namespace>
+        <remapping>image_raw:=/camera_front_left/image_raw</remapping>
+        <remapping>camera_info:=/camera_front_left/camera_info</remapping>
+      </ros>
+    </plugin>
+  </sensor>
+</gazebo>
+<!-- Back-right camera -->
+<gazebo reference="camera_back_right_link">
+  <sensor type="camera" name="camera_back_right_sensor">
+    <always_on>true</always_on>
+    <update_rate>30.0</update_rate>
+    <camera>
+      <horizontal_fov>1.047</horizontal_fov>
+      <image>
+        <width>640</width>
+        <height>480</height>
+        <format>R8G8B8</format>
+      </image>
+      <clip>
+        <near>0.02</near>
+        <far>50.0</far>
+      </clip>
+    </camera>
+    <plugin name="camera_back_right_controller" filename="libgazebo_ros_camera.so">
+      <ros>
+        <namespace>camera_back_right</namespace>
+        <remapping>image_raw:=/camera_back_right/image_raw</remapping>
+        <remapping>camera_info:=/camera_back_right/camera_info</remapping>
+      </ros>
+    </plugin>
+  </sensor>
+</gazebo>
+<!-- Back-left camera -->
+<gazebo reference="camera_back_left_link">
+  <sensor type="camera" name="camera_back_left_sensor">
+    <always_on>true</always_on>
+    <update_rate>30.0</update_rate>
+    <camera>
+      <horizontal_fov>1.047</horizontal_fov>
+      <image>
+        <width>640</width>
+        <height>480</height>
+        <format>R8G8B8</format>
+      </image>
+      <clip>
+        <near>0.02</near>
+        <far>50.0</far>
+      </clip>
+    </camera>
+    <plugin name="camera_back_left_controller" filename="libgazebo_ros_camera.so">
+      <ros>
+        <namespace>camera_back_left</namespace>
+        <remapping>image_raw:=/camera_back_left/image_raw</remapping>
+        <remapping>camera_info:=/camera_back_left/camera_info</remapping>
+      </ros>
+    </plugin>
+  </sensor>
+</gazebo>
 </robot>

File: rdsim_description/urdf/rdsim.urdf.xacro (robot description, xacro)
@@ -233,11 +233,36 @@
     <origin xyz="0.215 0 0.05" rpy="0 0 0"/>
   </joint>
-  <link name="camera_depth_frame"/>
-  <joint name="camera_depth_joint" type="fixed">
-    <origin xyz="0 0 0" rpy="${-pi/2} 0 ${-pi/2}"/>
-    <parent link="camera_link"/>
-    <child link="camera_depth_frame"/>
-  </joint>
-  <!-- Include gazebo macro -->
+  <!-- Add four cameras positioned diagonally at 45-degree angles -->
+  <xacro:macro name="add_camera" params="name x y z roll pitch yaw">
+    <link name="${name}_link">
+      <visual>
+        <origin xyz="0 0 0" rpy="0 0 0"/>
+        <geometry>
+          <box size="0.015 0.130 0.022"/>
+        </geometry>
+      </visual>
+      <collision>
+        <origin xyz="0 0 0" rpy="0 0 0"/>
+        <geometry>
+          <box size="0.015 0.130 0.022"/>
+        </geometry>
+      </collision>
+      <inertial>
+        <origin xyz="0 0 0" rpy="0 0 0"/>
+        <mass value="0.035"/>
+        <inertia ixx="0.001" ixy="0" ixz="0" iyy="0.001" iyz="0" izz="0.001"/>
+      </inertial>
+    </link>
+    <joint name="${name}_joint" type="fixed">
+      <parent link="base_link"/>
+      <child link="${name}_link"/>
+      <origin xyz="${x} ${y} ${z}" rpy="${roll} ${pitch} ${yaw}"/>
+    </joint>
+  </xacro:macro>
+  <!-- Adding four cameras in diagonal directions -->
+  <xacro:add_camera name="camera_front_right" x="0.25" y="0.25" z="0.25" roll="0" pitch="0" yaw="${pi/4}"/>
+  <xacro:add_camera name="camera_front_left" x="0.25" y="-0.25" z="0.25" roll="0" pitch="0" yaw="${-pi/4}"/>
+  <xacro:add_camera name="camera_back_right" x="-0.25" y="0.25" z="0.25" roll="0" pitch="0" yaw="${3*pi/4}"/>
+  <xacro:add_camera name="camera_back_left" x="-0.25" y="-0.25" z="0.25" roll="0" pitch="0" yaw="${-3*pi/4}"/>
   <xacro:include filename="$(find rdsim_description)/urdf/rdsim.gazebo.xacro" />
 </robot>

Commit message: feat : camera fov 장착 완료, fov 수정필요

File: rdsim_description/urdf/rdsim.gazebo.xacro (robot description, xacro)
@@ -268,8 +268,9 @@
 <gazebo reference="camera_front_right_link">
   <sensor type="camera" name="camera_front_right_sensor">
+    <visualize>${camera_visual}</visualize>
     <always_on>true</always_on>
     <update_rate>30.0</update_rate>
     <camera>
-      <horizontal_fov>1.047</horizontal_fov>
+      <horizontal_fov>1.347</horizontal_fov>
       <image>
         <width>640</width>
@@ -294,8 +295,9 @@
 <gazebo reference="camera_front_left_link">
   <sensor type="camera" name="camera_front_left_sensor">
+    <visualize>${camera_visual}</visualize>
     <always_on>true</always_on>
     <update_rate>30.0</update_rate>
     <camera>
-      <horizontal_fov>1.047</horizontal_fov>
+      <horizontal_fov>1.347</horizontal_fov>
       <image>
         <width>640</width>
@@ -320,8 +322,9 @@
 <gazebo reference="camera_back_right_link">
   <sensor type="camera" name="camera_back_right_sensor">
+    <visualize>${camera_visual}</visualize>
     <always_on>true</always_on>
     <update_rate>30.0</update_rate>
     <camera>
-      <horizontal_fov>1.047</horizontal_fov>
+      <horizontal_fov>1.347</horizontal_fov>
       <image>
         <width>640</width>
@@ -346,8 +349,9 @@
 <gazebo reference="camera_back_left_link">
   <sensor type="camera" name="camera_back_left_sensor">
+    <visualize>${camera_visual}</visualize>
     <always_on>true</always_on>
     <update_rate>30.0</update_rate>
     <camera>
-      <horizontal_fov>1.047</horizontal_fov>
+      <horizontal_fov>1.347</horizontal_fov>
       <image>
         <width>640</width>
@@ -369,3 +373,30 @@
   </sensor>
 </gazebo>
+<!-- camera_top_link -->
+<gazebo reference="camera_top_link">
+  <sensor type="camera" name="camera_top_sensor">
+    <visualize>${camera_visual}</visualize>
+    <always_on>true</always_on>
+    <update_rate>30.0</update_rate>
+    <camera>
+      <horizontal_fov>1.347</horizontal_fov>
+      <image>
+        <width>640</width>
+        <height>480</height>
+        <format>R8G8B8</format>
+      </image>
+      <clip>
+        <near>0.02</near>
+        <far>50.0</far>
+      </clip>
+    </camera>
+    <plugin name="camera_top_controller" filename="libgazebo_ros_camera.so">
+      <ros>
+        <namespace>camera_top</namespace>
+        <remapping>image_raw:=/camera_top/image_raw</remapping>
+        <remapping>camera_info:=/camera_top/camera_info</remapping>
+      </ros>
+    </plugin>
+  </sensor>
+</gazebo>
 </robot>

File: rdsim_description/urdf/rdsim.urdf.xacro (robot description, xacro)
@@ -242,15 +242,15 @@
         </geometry>
       </visual>
-      <collision>
+      <!-- <collision>
         <origin xyz="0 0 0" rpy="0 0 0"/>
         <geometry>
           <box size="0.015 0.130 0.022"/>
         </geometry>
-      </collision>
-      <inertial>
+      </collision> -->
+      <!-- <inertial>
         <origin xyz="0 0 0" rpy="0 0 0"/>
         <mass value="0.035"/>
         <inertia ixx="0.001" ixy="0" ixz="0" iyy="0.001" iyz="0" izz="0.001"/>
-      </inertial>
+      </inertial> -->
     </link>
     <joint name="${name}_joint" type="fixed">
@@ -265,4 +265,6 @@
   <xacro:add_camera name="camera_back_right" x="-0.25" y="0.25" z="0.25" roll="0" pitch="0" yaw="${3*pi/4}"/>
   <xacro:add_camera name="camera_back_left" x="-0.25" y="-0.25" z="0.25" roll="0" pitch="0" yaw="${-3*pi/4}"/>
+  <!-- top -->
+  <xacro:add_camera name="camera_top" x="0" y="0" z="5.25" roll="0" pitch="${pi/2}" yaw="0"/>
   <xacro:include filename="$(find rdsim_description)/urdf/rdsim.gazebo.xacro" />
 </robot>
